File: pcb/front-panel/front-panel.kicad_sch (KiCad schematic)
At the start: 0 parts

Commit message: Save
Parts:
- added RE1: RotaryEncoder_Switch, Rotary_Encoder:RotaryEncoder_Alps_EC11E-Switch_Vertical_H20mm, symbol Device:RotaryEncoder_Switch
- added U1: CC56-12SRWA, Display_7Segment:CA56-12SRWA, symbol Display_Character:CC56-12SRWA
- added U2: 74HC595, Package_SO:SOIC-16_3.9x9.9mm_P1.27mm, symbol 74xx:74HC595
Connections:
- new net GND: RE1.C, RE1.MP, RE1.S2
- new net RE1A: RE1.A
- new net RE1B: RE1.B
- new net RE1SW: RE1.S1
